File: electronics/freyja-gcs-pcb/design/freyja-gcs-pcb_nimmi.kicad_pcb (KiCad board)
At the start: 4 copper layers, 300 x 200 mm, 274 parts, among them J1 GT-USB-7010ASV, J10 XT60PB-M.G.Y, J11 XT60PB-F.G.Y, J2 JST SR, J3 2x20F, J4 JST SH, J5 JST SH, J6 GT-USB-7010ASV, J7 A2543WR-4P-2, J8 XD-PH-10AW, J9 JS350-S02DCA-00, Q1 TM10N06SI, Q10 NPN, Q11 NPN, Q12 NPN, Q13 NPN, Q14 NPN, Q15 NPN, Q16 NPN, Q17 NPN, Q18 NPN, Q19 NPN, Q2 TM10N06SI, Q20 NPN, Q21 NPN, Q22 NPN, Q23 NPN, Q24 AO4459, Q25 AO4459, Q3 AO4459, Q4 L2N7002SLLT1G, Q5 L2N7002SLLT1G, Q6 TM10N06SI, Q7 TM10N06SI, Q8 TM10N06SI, Q9 NPN, SW1 SW_SPST, SW10 PB22E09071, SW11 ST-0-102-A01-T000-LF+PJ, SW12 ST-0-102-A01-T000-LF+PJ, SW13 ST-0-102-A01-T000-LF+PJ, SW14 ST-0-102-A01-T000-LF+PJ, SW2 SW_SPST, SW3 K6-6136D-L1-04, SW4 PB22E09071, SW5 ST-0-102-A01-T000-LF+PJ, SW6 ST-0-102-A01-T000-LF+PJ, SW7 PB22E09071, SW8 ST-0-102-A01-T000-LF+PJ, SW9 ST-0-102-A01-T000-LF+PJ, U1 STM32U575RGTx, U10 LM74700QDBVRQ1, U11 AMS1117-3.3, U12 RY3730, U13 74HC595, U14 74HC595, U2 SN65HVD232DR, U3 FM7021DB, U4 CN3702, U5 HY2213-BB3A, U6 HY2213-BB3A, U7 IP2721, U8 SY8368AQQC, U9 LM74700QDBVRQ1, Y1 48MHz, Y2 32768Hz

Commit message: Updated PCB layout and grouped components
Parts:
- R69, R70, R71, R72, R73, R74, R75, R76: value 220 -> 560
- moved J6 332.4 mm to (270.0, 59.4), turned to 0 degrees
- moved R3 328.3 mm to (32.5, 130.0)
- moved R1 327.1 mm to (32.5, 125.0)
- moved C17 317.7 mm to (28.5, 137.5), turned to 0 degrees
- moved R2 308.1 mm to (32.5, 127.5), turned to 0 degrees
- moved D3 303.8 mm to (53.0, 86.7)
- moved R79 299.8 mm to (54.2, 125.5)
- moved D1 299.0 mm to (53.0, 81.5)
- moved D6 296.3 mm to (57.4, 84.1)
- moved D4 294.3 mm to (53.0, 89.3)
- moved D2 291.7 mm to (53.0, 84.1)
- moved D8 290.2 mm to (57.4, 89.3)
- moved D7 289.8 mm to (57.4, 86.7)
- moved D9 287.7 mm to (68.5, 73.5)
- moved R75 251.5 mm to (192.5, 2.15), turned to 0 degrees
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Connections:
- C45 pad 2: +3V3 -> +5V
- C46 pad 1: +3V3 -> +5V
- C47 pad 2: +3V3 -> +5V
- C48 pad 1: +3V3 -> +5V
- Q24 pad 1: +3V3 -> Net-(Q24-S-Pad1)
- Q24 pad 2: +3V3 -> Net-(Q24-S-Pad1)
- Q24 pad 3: +3V3 -> Net-(Q24-S-Pad1)
- Q25 pad 1: +3V3 -> Net-(Q25-S-Pad1)
- Q25 pad 2: +3V3 -> Net-(Q25-S-Pad1)
- Q25 pad 3: +3V3 -> Net-(Q25-S-Pad1)
- R67 pad 2: +3V3 -> +5V
- R68 pad 2: +3V3 -> +5V
- U13 pad 16: +3V3 -> +5V
- U14 pad 16: +3V3 -> +5V
Other:
- board outline removed
