File: electronics/freyja-gcs-pcb/design/freyja-gcs-pcb.kicad_pcb (KiCad board)
At the start: 4 copper layers, 300 x 200 mm, 274 parts, among them J1 GT-USB-7010ASV, J10 XT60PB-M.G.Y, J11 XT60PB-F.G.Y, J2 JST SR, J3 2x20F, J4 JST SH, J5 JST SH, J6 GT-USB-7010ASV, J7 A2543WR-4P-2, J8 XD-PH-10AW, J9 JS350-S02DCA-00, Q1 TM10N06SI, Q10 NPN, Q11 NPN, Q12 NPN, Q13 NPN, Q14 NPN, Q15 NPN, Q16 NPN, Q17 NPN, Q18 NPN, Q19 NPN, Q2 TM10N06SI, Q20 NPN, Q21 NPN, Q22 NPN, Q23 NPN, Q24 AO4459, Q25 AO4459, Q3 AO4459, Q4 L2N7002SLLT1G, Q5 L2N7002SLLT1G, Q6 TM10N06SI, Q7 TM10N06SI, Q8 TM10N06SI, Q9 NPN, SW1 SW_SPST, SW10 PB22E09071, SW11 ST-0-102-A01-T000-LF+PJ, SW12 ST-0-102-A01-T000-LF+PJ, SW13 ST-0-102-A01-T000-LF+PJ, SW14 ST-0-102-A01-T000-LF+PJ, SW2 SW_SPST, SW3 K6-6136D-L1-04, SW4 PB22E09071, SW5 ST-0-102-A01-T000-LF+PJ, SW6 ST-0-102-A01-T000-LF+PJ, SW7 PB22E09071, SW8 ST-0-102-A01-T000-LF+PJ, SW9 ST-0-102-A01-T000-LF+PJ, U1 STM32U575RGTx, U10 LM74700QDBVRQ1, U11 AMS1117-3.3, U12 RY3730, U13 74HC595, U14 74HC595, U2 SN65HVD232DR, U3 FM7021DB, U4 CN3702, U5 HY2213-BB3A, U6 HY2213-BB3A, U7 IP2721, U8 SY8368AQQC, U9 LM74700QDBVRQ1, Y1 48MHz, Y2 32768Hz

Commit message: PCB rough design layout - COMPLETED
Parts:
- BT2, BT3, BT4, BT5: moved to B.Cu
- moved BT3 196.7 mm to (130.0, 41.7), turned to 90 degrees
- moved C2 190.4 mm to (258.5, 62.3)
- moved Y2 189.8 mm to (260.9, 60.5)
- moved C4 188.4 mm to (263.3, 62.3)
- moved C6 182.1 mm to (246.2, 94.2)
- moved Q23 181.7 mm to (256.8, 127.1), turned to 90 degrees
- moved D46 176.5 mm to (50.1, 148.0)
- moved R55 176.5 mm to (44.3, 148.0)
- moved SW10 176.5 mm to (47.1, 140.7)
- moved D5 170.5 mm to (234.2, 93.4)
- moved D57 169.2 mm to (258.6, 131.0)
- moved C16 165.4 mm to (275.9, 68.8), turned to -90 degrees
- moved R66 164.4 mm to (259.7, 127.1)
- moved R8 164.2 mm to (274.3, 65.2), turned to -90 degrees
- moved D11 162.7 mm to (272.8, 68.7), turned to -90 degrees
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Other:
- board size 300 x 200 mm -> 301 x 200 mm

Commit message: Updated edge cuts, added holes, curved edges, rearranged LEDs, moved battries to top, changed the power delivery USB to right side.
Parts:
- added H5: M2.5 12mm, EasyEDA:SMTSO25, F.Cu at (4.50, 4.90)
- added H6: M2.5 12mm, EasyEDA:SMTSO25, F.Cu at (4.50, 195.7)
- added H7: M2.5 12mm, EasyEDA:SMTSO25, F.Cu at (222.3, 85.3)
- added H8: M2.5 12mm, EasyEDA:SMTSO25, F.Cu at (224.8, 194.1)
- added R81: 10k, Resistor_SMD:R_0603_1608Metric, F.Cu at (8.53, 2.70)
- added R82: 10k, Resistor_SMD:R_0603_1608Metric, F.Cu at (8.88, 193.5)
- added R83: 10k, Resistor_SMD:R_0603_1608Metric, F.Cu at (225.6, 82.5)
- added R84: 10k, Resistor_SMD:R_0603_1608Metric, F.Cu at (224.2, 190.6)
- BT2, BT3, BT4, BT5: moved to F.Cu
- moved J6 311.1 mm to (295.7, 119.3), turned to 90 degrees
- moved D19 304.3 mm to (290.1, 123.8), turned to 180 degrees
- moved D15 302.1 mm to (290.2, 120.7), turned to 180 degrees
- moved R20 300.6 mm to (290.2, 118.8), turned to 0 degrees
- moved D16 297.6 mm to (290.1, 114.8), turned to 180 degrees
- moved C23 296.9 mm to (286.0, 124.1), turned to -90 degrees
- moved R26 291.3 mm to (282.9, 124.1), turned to -90 degrees
- moved Q6 289.7 mm to (287.1, 111.7), turned to 90 degrees
- moved U7 288.5 mm to (283.6, 119.0), turned to 90 degrees
- moved R19 288.2 mm to (281.2, 124.0), turned to 90 degrees
- moved F1 271.9 mm to (276.6, 114.2), turned to 90 degrees
- moved C26 271.6 mm to (273.2, 121.5), turned to 180 degrees
- moved C25 251.9 mm to (242.4, 153.1)
- moved R25 251.9 mm to (242.2, 146.9)
- moved R27 251.9 mm to (257.4, 152.0)
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Other:
- board size 301 x 200 mm -> 300 x 200 mm

Commit message: power layout wip
Parts:
- added H10: M2.5 12mm, EasyEDA:SMTSO25, F.Cu at (318.0, 218.0)
- added H9: M2.5 12mm, EasyEDA:SMTSO25, F.Cu at (297.0, 26.0)
- added R85: 10k, Resistor_SMD:R_0603_1608Metric, F.Cu at (291.5, 26.0)
- added R86: 10k, Resistor_SMD:R_0603_1608Metric, F.Cu at (312.5, 218.0)
- C29: value 100n -> 22u; footprint Capacitor_SMD:C_0603_1608Metric -> EasyEDA:C1210
- moved R27 102.6 mm to (158.3, 125.0)
- moved C19 102.6 mm to (134.8, 115.5)
- moved C20 102.6 mm to (132.8, 126.3)
- moved C24 102.6 mm to (143.4, 123.2)
- moved C25 102.6 mm to (143.4, 126.1)
- moved D13 102.6 mm to (138.4, 110.0)
- moved D14 102.6 mm to (151.4, 125.6)
- moved D17 102.6 mm to (149.0, 121.4)
- moved D18 102.6 mm to (156.3, 120.2)
- moved L1 102.6 mm to (157.4, 109.9)
- moved Q3 102.6 mm to (145.0, 113.2)
- moved R12 102.6 mm to (147.5, 126.1)
- moved R13 102.6 mm to (132.6, 119.6)
- moved R14 102.6 mm to (134.8, 112.5)
- moved R15 102.6 mm to (138.8, 115.9)
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Connections:
- C29 pad 1: /Power/VPWR -> +5V
Routing:
- net Net-(D21-K): track 0.00 -> 26.8 mm, vias 0 -> 2
- net +5V: track 0.00 -> 20.5 mm, vias 0 -> 2
- net Net-(U8-BS): track 0.00 -> 11.0 mm, vias 0 -> 2
- net Net-(D30-K): track 0.00 -> 10.4 mm, vias 0 -> 2
- net Net-(U8-ILMT): track 0.00 -> 5.82 mm, vias 0 -> 2
- net Net-(U8-LX): track 0.00 -> 3.62 mm
- net Net-(U8-EN): track 0.00 -> 1.50 mm, vias 0 -> 1
- net Net-(D26-A): track 0.00 -> 1.38 mm
- net Net-(D21-A): track 0.00 -> 1.38 mm
- net Net-(D29-A1): track 0.00 -> 1.14 mm, vias 0 -> 1
- net GND: vias 0 -> 24
- net (no net): vias 0 -> 1
- added copper zone on F.Cu, net +5V
- added copper zone on F.Cu, net /Power/VPWR
- added copper zone on F.Cu, net Net-(D30-A)
- added copper zone on F.Cu, net Net-(D30-K)
- added copper zone on F.Cu, net Net-(U12-FB)
- added copper zone on F.Cu, net Net-(U8-FB)
- added copper zone on F.Cu, net Net-(U8-LX)
- added copper zone on F.Cu, net Net-(U8-VCC)
Other:
- outline, holes or cut-outs redrawn

Commit message: locked position of components
Parts:
- added D58: Green, EasyEDA:LED-TH_BD5.9-P2.54-RD_GREEN, F.Cu at (167.0, 162.0)
- added H11: M2.5 12mm, EasyEDA:SMTSO25, F.Cu at (26.0, 122.0)
- added H12: M2.5 12mm, EasyEDA:SMTSO25, F.Cu at (172.0, 122.0)
- added H13: M2.5 12mm, EasyEDA:SMTSO25, F.Cu at (318.0, 122.0)
- added Q26: NPN, EasyEDA:SOT-416_L1.6-W0.8-P1.00-LS1.6-BR, F.Cu at (172.0, 160.0)
- added R87: 10k, Resistor_SMD:R_0603_1608Metric, F.Cu at (31.5, 122.0)
- added R88: 10k, Resistor_SMD:R_0603_1608Metric, F.Cu at (166.5, 122.0)
- added R89: 10k, Resistor_SMD:R_0603_1608Metric, F.Cu at (312.0, 122.0)
- added R90: 220, Resistor_SMD:R_0603_1608Metric, F.Cu at (172.0, 162.0)
- D56: value Yellow -> Green
- moved R63 68.5 mm to (172.0, 142.0), turned to 180 degrees
- moved Q20 68.5 mm to (172.0, 140.0), turned to 0 degrees
- moved D54 63.8 mm to (167.0, 142.0)
- moved D52 57.3 mm to (167.0, 132.0)
- moved D53 55.0 mm to (107.0, 142.0)
- moved TP5 53.9 mm to (192.0, 57.0)
- moved C31 53.8 mm to (172.1, 55.9)
- moved C34 53.8 mm to (171.9, 51.6)
- moved C35 53.8 mm to (172.7, 63.9)
- moved D20 53.8 mm to (168.3, 56.9)
- moved TP2 53.8 mm to (176.9, 46.4)
- moved C30 53.8 mm to (172.5, 58.8)
- moved C32 53.8 mm to (171.9, 48.7)
- moved C33 53.8 mm to (172.8, 60.7)
- moved Q7 53.8 mm to (181.2, 53.2)
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Connections:
- C43 pad 1: +3.3V -> +3V3
- D25 pad 2: +3.3V -> +3V3
- D27 pad 1: +3.3V -> +3V3
- Q22 pad 1: AUX_LED -> AUX1_LED
- R38 pad 1: +3.3V -> +3V3
- TP8 pad 1: +3.3V -> +3V3
- U1 pad 23: unconnected-(U1-PA7-Pad23) -> LAUNCH_ARMD
- U1 pad 26: AUX_BTN -> LAUNCH_ARMD_LED
- U1 pad 27: LAUNCH_ARMD_LED -> CMD_ARMD_LED
- U1 pad 28: CMD_ARMD_LED -> FAULT_LED
- U1 pad 29: AUX_LED -> AUX2_LED
- U1 pad 41: LAUNCH_ARMD -> LAUNCH
- U1 pad 42: LAUNCH -> CMD_ARMD
- U1 pad 43: CMD_ARMD -> CMD_SEND
- U1 pad 50: CMD_SEND -> AUX_BTN
- U1 pad 55: FAULT_LED -> CON_STS_RKT
- U1 pad 56: CON_STS_RKT -> CON_STS_LPD
- U1 pad 57: CON_STS_LPD -> LAUNCHED_LED
- U1 pad 59: LAUNCHED_LED -> AUX1_LED
- U11 pad 2: +3.3V -> +3V3
Routing:
- net GND: track 0.00 -> 108.7 mm, vias 24 -> 83
- net Net-(U8-EN): track 1.50 -> 45.5 mm, vias 1 -> 2
- net +5V: track 20.5 -> 60.7 mm
- net CMD_ARMD: track 0.00 -> 25.5 mm
- net LAUNCH_ARMD: track 0.00 -> 24.5 mm
- net Net-(SW3-+): track 0.00 -> 7.07 mm
- net Net-(D58-K): track 0.00 -> 6.45 mm
- net Net-(D56-K): track 0.00 -> 6.45 mm
- net Net-(D54-K): track 0.00 -> 6.45 mm
- net Net-(D52-K): track 0.00 -> 6.45 mm
- net Net-(D57-K): track 0.00 -> 6.45 mm
- net Net-(D55-K): track 0.00 -> 6.45 mm
- net Net-(D53-K): track 0.00 -> 6.45 mm
- net Net-(D51-K): track 0.00 -> 6.45 mm
- net TGL6: track 0.00 -> 6.08 mm
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- added copper zone on In2.Cu, net +3V3
- added copper zone on F.Cu, net GND
- added copper zone on In1.Cu, net GND
- added copper zone on F.Cu, net Net-(BT2--)
- added copper zone on F.Cu, net Net-(BT4--)

Commit message: mcu layout
Parts:
- added D59: PSBD1DF40V2L, EasyEDA:SOD-123FL_L2.8-W1.8-LS3.8-RD, F.Cu at (277.0, 92.0)
- moved BT1 113.9 mm to (362.7, 113.6)
- moved D5 113.9 mm to (356.3, 122.7)
- moved TP2 81.9 mm to (220.0, 116.0)
- moved D20 76.0 mm to (204.0, 124.0)
- moved TP3 70.9 mm to (201.0, 136.3)
- moved C31 69.3 mm to (209.0, 114.5), turned to -90 degrees
- moved C32 67.2 mm to (189.7, 113.5), turned to 0 degrees
- moved C33 64.0 mm to (207.5, 114.5), turned to 90 degrees
- moved C34 61.6 mm to (188.2, 111.0), turned to -90 degrees
- moved C35 61.3 mm to (205.0, 116.0), turned to 0 degrees
- moved Q7 60.0 mm to (197.2, 111.0)
- moved U9 59.9 mm to (191.7, 111.0)
- moved C30 58.8 mm to (189.7, 115.0), turned to 180 degrees
- moved C43 58.6 mm to (270.0, 96.0), turned to 0 degrees
- moved U10 58.1 mm to (205.0, 112.5), turned to 0 degrees
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Connections:
- net VBUS renamed VBUS_DEV
- C34 pad 1: Net-(U9-EN) -> Net-(U9-VCAP)
- C35 pad 1: Net-(U10-EN) -> Net-(U10-VCAP)
- D2 pad 1: Net-(D2-A1) -> /USB_D_P
- J1 pad A6: Net-(D2-A1) -> /USB_D_P
- J1 pad B6: Net-(D2-A1) -> /USB_D_P
- J2 pad MP: unconnected-(J2-PadMP)_1 -> GND
- U10 pad 1: Net-(U10-EN) -> Net-(U10-VCAP)
- U10 pad 3: Net-(U10-EN) -> /Power/VBAT
- U9 pad 1: Net-(U9-EN) -> Net-(U9-VCAP)
- U9 pad 3: Net-(U9-EN) -> /Power/VBUS
Routing:
- net /BOOT0: track 0.00 -> 74.9 mm, vias 0 -> 2
- net GND: track 108.7 -> 179.7 mm, vias 83 -> 123
- net NRST: track 0.00 -> 68.8 mm, vias 0 -> 2
- net VBUS_DEV: track 0.00 -> 60.6 mm, vias 0 -> 7
- net +5V: track 60.7 -> 98.3 mm
- net /SWCLK: track 0.00 -> 37.1 mm, vias 0 -> 2
- net /USB_D_N: track 0.00 -> 35.5 mm
- net /USB_D_P: track 0.00 -> 35.5 mm
- net +3V3: track 0.00 -> 33.1 mm, vias 0 -> 9
- net /SWDIO: track 0.00 -> 32.8 mm, vias 0 -> 2
- net /Power/VBAT: track 0.00 -> 14.6 mm, vias 0 -> 12
- net Net-(J2-Pin_1): track 0.00 -> 8.34 mm
- net Net-(U1-PC14): track 0.00 -> 8.28 mm
- net Net-(U1-PC15): track 0.00 -> 8.06 mm
- net Net-(U1-PH1): track 0.00 -> 7.20 mm
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- added copper zone on F.Cu, net +3V3
- added copper zone on F.Cu, net /Power/BAT-
- added copper zone on F.Cu, net /Power/VBAT

Commit message: usb pd layout
Parts:
- added D60: PESD2IVN24-TR, EasyEDA:TO-236AB_L2.9-W1.3-P0.95-LS2.3-BR, F.Cu at (307.0, 154.6)
- moved Q1 25.0 mm to (162.4, 61.2)
- moved R11 25.0 mm to (167.3, 57.8)
- moved R22 25.0 mm to (170.2, 50.0)
- moved R23 25.0 mm to (157.7, 63.5)
- moved R24 25.0 mm to (167.0, 50.0)
- moved TP1 25.0 mm to (175.8, 47.0)
- moved U3 25.0 mm to (169.6, 53.6)
- moved U5 25.0 mm to (169.8, 62.1)
- moved C21 25.0 mm to (173.7, 61.8)
- moved C22 25.0 mm to (173.7, 50.7)
- moved Q2 25.0 mm to (162.1, 53.3)
- moved R21 25.0 mm to (157.6, 60.3)
- moved U6 25.0 mm to (156.5, 51.8)
- moved C30 21.3 mm to (211.0, 114.0), turned to -90 degrees
- moved C32 19.8 mm to (209.5, 114.0), turned to 90 degrees
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Routing:
- net Net-(BT4--): track 0.00 -> 101.9 mm
- net Net-(BT2--): track 0.00 -> 101.9 mm
- net /Power/VBUS: track 5.50 -> 104.4 mm, vias 0 -> 18
- net Net-(Q6-D): track 0.00 -> 40.3 mm
- net /Power/BAT-: track 0.00 -> 23.3 mm
- net GND: track 179.7 -> 200.9 mm, vias 123 -> 136
- net Net-(D19-A1): track 0.00 -> 19.9 mm, vias 0 -> 2
- net Net-(D15-A1): track 0.00 -> 19.3 mm, vias 0 -> 2
- net Net-(D16-A1): track 0.00 -> 17.2 mm, vias 0 -> 2
- net Net-(Q6-S): track 0.00 -> 12.5 mm, vias 0 -> 2
- net Net-(U7-SEL): track 0.00 -> 6.97 mm
- net +5V: track 98.3 -> 103.7 mm
- net +3V3: track 33.1 -> 37.6 mm, vias 9 -> 13
- net /Power/VBAT: vias 12 -> 9
- added copper zone on F.Cu, net /Power/VBUS
- added copper zone on F.Cu, net Net-(Q6-S)
- removed copper zone on F.Cu, net /Power/BAT-
- removed copper zone on F.Cu, net Net-(BT2--)
- removed copper zone on F.Cu, net Net-(BT4--)

Commit message: charging circuit layout wip
Parts:
- added C49: 22u, EasyEDA:C2220, F.Cu at (146.5, 72.5)
- added TP10: TestPoint, TestPoint:TestPoint_Pad_D3.0mm, F.Cu at (146.0, 91.0)
- C20: value 100n -> 470n
- moved Q2 67.4 mm to (129.0, 112.0), turned to 90 degrees
- moved R14 67.2 mm to (75.2, 72.1)
- moved TP1 63.4 mm to (146.0, 103.0)
- moved U3 60.6 mm to (134.5, 103.0), turned to -90 degrees
- moved R22 59.7 mm to (136.0, 99.0), turned to 90 degrees
- moved Q1 57.7 mm to (135.0, 112.0), turned to 90 degrees
- moved C22 56.1 mm to (137.5, 93.5), turned to -90 degrees
- moved D14 55.5 mm to (155.6, 56.3)
- moved R12 55.5 mm to (151.6, 56.8)
- moved R11 55.1 mm to (138.0, 104.5), turned to 180 degrees
- moved D13 55.0 mm to (142.5, 41.2)
- moved R15 55.0 mm to (142.9, 47.1)
- moved R16 51.5 mm to (148.7, 59.4)
- moved C20 49.8 mm to (151.8, 65.5), turned to 90 degrees
- moved R24 48.9 mm to (137.5, 89.0), turned to -90 degrees
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Connections:
- BT4 pad 1: Net-(BT4--) -> Net-(BT2--)
- BT5 pad 2: Net-(BT4--) -> Net-(BT2--)
- C21 pad 2: Net-(BT4--) -> Net-(BT2--)
- Q4 pad 2: Net-(BT4--) -> Net-(BT2--)
- R11 pad 2: /Power/BAT- -> Net-(U3-CS)
- R22 pad 2: Net-(BT4--) -> Net-(BT2--)
- R24 pad 1: Net-(BT4--) -> Net-(BT2--)
- R29 pad 1: Net-(BT4--) -> Net-(BT2--)
- U3 pad 3: unconnected-(U3-CS-Pad3) -> Net-(U3-CS)
- U5 pad 3: Net-(BT4--) -> Net-(BT2--)
Routing:
- net /Power/VBAT: track 14.6 -> 211.2 mm, vias 9 -> 22
- net Net-(BT2--): track 101.9 -> 216.6 mm
- net Net-(BT4--): track 101.9 -> 0.00 mm
- net /Power/VBUS: track 104.4 -> 184.9 mm, vias 18 -> 27
- net /Power/BAT-: track 23.3 -> 61.9 mm
- net Net-(Q5-G): track 0.00 -> 12.1 mm
- net Net-(Q4-G): track 0.00 -> 12.1 mm
- net Net-(Q2-G): track 0.00 -> 7.86 mm
- net Net-(Q1-G): track 0.00 -> 7.12 mm
- net GND: track 200.9 -> 208.0 mm, vias 136 -> 149
- net Net-(U4-CSP): track 0.00 -> 6.23 mm
- net Net-(U4-EOC): track 0.00 -> 4.92 mm
- net Net-(U6-VDD): track 0.00 -> 4.66 mm
- net Net-(U5-VDD): track 0.00 -> 4.66 mm
- net Net-(Q3-G): track 0.00 -> 3.98 mm
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- added copper zone on F.Cu, net /Power/BAT-
- added copper zone on F.Cu, net Net-(D17-A)
- added copper zone on F.Cu, net Net-(D17-K)
- added copper zone on F.Cu, net Net-(Q1-D)
- added copper zone on F.Cu, net Net-(U4-CSP)
