File: electronics/freyja-gcs-pcb/design/freyja-gcs-pcb.kicad_pcb (KiCad board)
At the start: 4 copper layers, 300 x 200 mm, 299 parts, among them J1 GT-USB-7010ASV, J10 XT60PB-M.G.Y, J11 XT60PB-F.G.Y, J2 JST SR, J3 2x20F, J4 JST SH, J5 JST SH, J6 GT-USB-7010ASV, J7 A2543WR-4P-2, J8 XD-PH-10AW, J9 JS350-S02DCA-00, Q1 TM10N06SI, Q10 NPN, Q11 NPN, Q12 NPN, Q13 NPN, Q14 NPN, Q15 NPN, Q16 NPN, Q17 NPN, Q18 NPN, Q19 NPN, Q2 TM10N06SI, Q20 NPN, Q21 NPN, Q22 NPN, Q23 NPN, Q24 AO4459, Q25 AO4459, Q26 NPN, Q3 AO4459, Q4 L2N7002SLLT1G, Q5 L2N7002SLLT1G, Q6 TM10N06SI, Q7 TM10N06SI, Q8 TM10N06SI, Q9 NPN, SW1 SW_SPST, SW10 PB22E09071, SW11 ST-0-102-A01-T000-LF+PJ, SW12 ST-0-102-A01-T000-LF+PJ, SW13 ST-0-102-A01-T000-LF+PJ, SW14 ST-0-102-A01-T000-LF+PJ, SW2 SW_SPST, SW3 K6-6136D-L1-04, SW4 PB22E09071, SW5 ST-0-102-A01-T000-LF+PJ, SW6 ST-0-102-A01-T000-LF+PJ, SW7 PB22E09071, SW8 ST-0-102-A01-T000-LF+PJ, SW9 ST-0-102-A01-T000-LF+PJ, U1 STM32U575RGTx, U10 LM74700QDBVRQ1, U11 AMS1117-3.3, U12 RY3730, U13 74HC595, U14 74HC595, U2 SN65HVD232DR, U3 FM7021DB, U4 CN3702, U5 HY2213-BB3A, U6 HY2213-BB3A, U7 IP2721, U8 SY8368AQQC, U9 LM74700QDBVRQ1, Y1 48MHz, Y2 32768Hz

Commit message: all routed, fine tuning left
Parts:
- added C50: 100n, Capacitor_SMD:C_0603_1608Metric, F.Cu at (50.0, 179.4)
- added C51: 100n, Capacitor_SMD:C_0603_1608Metric, F.Cu at (114.8, 133.1)
- added C52: 100n, Capacitor_SMD:C_0603_1608Metric, F.Cu at (174.7, 133.1)
- added C53: 100n, Capacitor_SMD:C_0603_1608Metric, F.Cu at (133.0, 57.0)
- added C54: 100n, Capacitor_SMD:C_0603_1608Metric, F.Cu at (158.8, 60.5)
- moved D59 16.0 mm to (293.0, 91.5)
Connections:
- net /Power/VBUS renamed VBUS
Routing:
- net +5V: track 109.2 -> 711.6 mm, vias 2 -> 26
- net VBUS_DEV: track 60.6 -> 46.0 mm
- net GND: track 239.4 -> 246.0 mm, vias 173 -> 179
- net /CAN_RX: track 46.7 -> 48.7 mm
- net /CAN_TX: track 49.6 -> 51.3 mm

Commit message: cleanup
Parts:
- H1, H2, H3, H4: footprint EasyEDA:SMTSO25 -> EasyEDA:SMTSO25120
- H10, H11, H12, H13, H5, H6, H7, H8, H9: footprint EasyEDA:SMTSO25 -> EasyEDA:SMTSO25100
- moved R87 7.94 mm to (31.5, 122.1), turned to 0 degrees
- moved TP5 6.02 mm to (207.0, 98.0)
- moved TP6 6.00 mm to (230.5, 74.0)
- turned R78 to 180 degrees
Connections:
- net /Power/BAT- renamed /Power/NBAT
- net Net-(BT2--) renamed /Power/MBAT
Routing:
- net GND: track 246.0 -> 250.2 mm, vias 179 -> 182
- net +5V: track 711.6 -> 708.1 mm
- net TGL0: track 270.2 -> 271.4 mm
- net /BOOT0: track 76.6 -> 77.8 mm

Commit message: aesir logo
Parts:
- added G***: LOGO, prjlib:aesir_logo_large, F.Cu at (241.0, 127.0)

Commit message: annotation and pinouts
Parts:
- added G***: LOGO, prjlib:euroc_logo, B.Cu at (172.0, 122.0)
- moved G*** 20.2 mm to (221.0, 124.0)
Other:
- board text added: "+"
- board text added: "-"
- board text added: "12V"
- board text added: "3V3"
- board text added: "5V"
- board text added: "5V PWRON"
- board text added: "9-20V PD"
- board text added: "ADJ"
- board text added: "AUX BTN"
- board text added: "BACKLIGHT PWR"
- board text added: "CAN"
- board text added: "CHARGE USB"
- board text added: "CMD SEND"
- board text added: "CMD SEND ARM"
- board text added: "CR2032 RTC BAT"
- board text added: "FAN 5V"
- board text added: "FREYJA GROUND CONTROL STATION"
- board text added: "GND"
- board text added: "H"
- board text added: "HUGO FRISK SRI NIRMAL KUMAAR"
- board text added: "L"
- board text added: "LAUNCH"
- board text added: "LAUNCH ARM"
- board text added: "LCD BACKLIGHT"
- board text added: "LCD DRIVER POWER"
- board text added: "MBAT"
- board text added: "MCU USB"
- board text added: "NBAT"
- board text added: "NC"
- board text added: "PWM"
- board text added: "REV 1.0 EUROC 25"
- board text added: "SWD"
- board text added: "TAC"
- board text added: "TEMP"
- board text added: "VBAT"
- board text added: "VBUS"
- board text added: "VPWR"
